File: Ethernet_W5500.sch (KiCad schematic (older format))
At the start: 1 part

Commit message: Upd
Parts:
- added C1: 22n, Capacitors_SMD:C_0805, symbol C_Cer_SMD_0805
- added C10, C12, C13, C14, C15, C16, C18: 100n, Capacitors_SMD:C_0805, symbol C_Cer_SMD_0805
- added C11, C17: 10u, Capacitors_SMD:C_1206, symbol C_Cer_SMD_1206
- added C2, C3: 6.8n, Capacitors_SMD:C_0805, symbol C_Cer_SMD_0805
- added C4, C9: 10n, Capacitors_SMD:C_0805, symbol C_Cer_SMD_0805
- added C5: 1n/2KV, Capacitors_SMD:C_1206, symbol C_Cer_SMD_1206
- added C6, C7: 18p, Capacitors_SMD:C_0805, symbol C_Cer_SMD_0805
- added C8: 4.7u, Capacitors_SMD:C_0805, symbol C_Cer_SMD_0805
- added FB1: 120, Resistors_SMD:R_0805, symbol FB_SMD_0805
- added R1, R2, R3, R8, R9: 49R9, Resistors_SMD:R_0805, symbol R_SMD_0805
- added R10: 1M, Resistors_SMD:R_0805, symbol R_SMD_0805
- added R11, R12: 330, Resistors_SMD:R_0805, symbol R_SMD_0805
- added R13: 12.4K 1%, Resistors_SMD:R_0805, symbol R_SMD_0805
- added R4, R5, R6, R7: 33, Resistors_SMD:R_0805, symbol R_SMD_0805
- added U1: HR911105A, RJ45ALED_1PRIMARY, symbol HR911105A
- added X1: 25Mhz, BK_Common:crystal_smd_3225_4pin, symbol Chrystal_SMD_3225_4pin
- gave numbers to parts that had none: 1
Connections:
- net labels added: +3.3VADC, +3V3, ACTLED, GND, INTn, LNKLED, MOSI, RSTn, RXN, RXP, SCLK, SCSn, TXN, TXP, VDD_3V3
- wire segments 0 -> 133
- no-connect marks 0 -> 4
Other:
- moved on the sheet: U2
