File: RS_485_3V3.sch (KiCad schematic (older format))
At the start: 3 parts

Commit message: Upd
Parts:
- added J2, J3: RJ12, BK_Common:RJ12_2mm_Pitch, symbol RJ12
- added R15, R17, R20: 10K, Resistors_SMD:R_0805, symbol R_SMD_0805
- added R16, R19, R22: 20K, Resistors_SMD:R_0805, symbol R_SMD_0805
- added R18, R21: 120, Resistors_SMD:R_0805, symbol R_SMD_0805
- added U4, U5: MAX487, Housings_SOIC:SOIC-8_3.9x4.9mm_Pitch1.27mm, symbol MAX487
- gave numbers to parts that had none: 3
Connections:
- net labels added: 485_A1, 485_A2, 485_A3, 485_B1, 485_B2, 485_B3, DE_O1, DE_O2, DE_O3, RxD1, RxD2, RxD3, TxD1, TxD2, TxD3
- net labels removed: 485_A, 485_B, DE_O, RxD, TxD
- wire segments 28 -> 88
- no-connect marks 0 -> 12
Other:
- moved on the sheet: J1
