File: Room_Controller.kicad_pcb (KiCad board)
At the start: 2 copper layers, 101.6 x 53.3 mm, 14 parts, among them P1 Digital, P10 CONN_1, P11 CONN_1, P12 CONN_1, P13 CONN_1, P14 ICSP, P2 Power, P3 Analog, P4 Analog, P5 PWM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

Commit message: Upd
Other:
- board size 101.6 x 53.3 mm -> 99 x 53.3 mm
Changed lines of the file:
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@@
     (links 9)
     (no_connects 9)
-    (area 103.302999 68.250999 205.053001 121.741001)
+    (area 96.952999 66.693 205.053001 122.895)
     (thickness 1.6)
-    (drawings 27)
+    (drawings 28)
     (tracks 0)
     (zones 0)
@@
     )
   )
+  (gr_line (start 202.378 68.326) (end 202.378 70.866) (angle 90) (layer Edge.Cuts) (width 0.15))
   (gr_text 1 (at 131.318 116.586 90) (layer F.SilkS)
     (effects (font (size 1 1) (thickness 0.15)))
@@
   (gr_line (start 114.808 109.601) (end 114.808 118.491) (angle 90) (layer Dwgs.User) (width 0.15))
   (gr_line (start 101.473 109.601) (end 114.808 109.601) (angle 90) (layer Dwgs.User) (width 0.15))
-  (gr_line (start 202.438 121.666) (end 103.378 121.666) (angle 90) (layer Edge.Cuts) (width 0.15))
-  (gr_line (start 202.438 120.396) (end 202.438 121.666) (angle 90) (layer Edge.Cuts) (width 0.15))
-  (gr_line (start 204.978 117.856) (end 202.438 120.396) (angle 90) (layer Edge.Cuts) (width 0.15))
-  (gr_line (start 204.978 83.566) (end 204.978 117.856) (angle 90) (layer Edge.Cuts) (width 0.15))
-  (gr_line (start 202.438 81.026) (end 204.978 83.566) (angle 90) (layer Edge.Cuts) (width 0.15))
-  (gr_line (start 202.438 70.866) (end 202.438 81.026) (angle 90) (layer Edge.Cuts) (width 0.15))
-  (gr_line (start 199.898 68.326) (end 202.438 70.866) (angle 90) (layer Edge.Cuts) (width 0.15))
+  (gr_line (start 202.378 121.666) (end 103.378 121.666) (angle 90) (layer Edge.Cuts) (width 0.15))
+  (gr_line (start 202.378 120.396) (end 202.378 121.666) (angle 90) (layer Edge.Cuts) (width 0.15))
+  (gr_line (start 202.378 117.856) (end 202.378 120.396) (angle 90) (layer Edge.Cuts) (width 0.15))
+  (gr_line (start 202.378 83.566) (end 202.378 117.856) (angle 90) (layer Edge.Cuts) (width 0.15))
+  (gr_line (start 202.378 81.026) (end 202.378 83.566) (angle 90) (layer Edge.Cuts) (width 0.15))
+  (gr_line (start 202.378 70.866) (end 202.378 81.026) (angle 90) (layer Edge.Cuts) (width 0.15))
+  (gr_line (start 199.898 68.326) (end 202.378 68.326) (angle 90) (layer Edge.Cuts) (width 0.15))
   (gr_line (start 103.378 68.326) (end 199.898 68.326) (angle 90) (layer Edge.Cuts) (width 0.15))
   (gr_line (start 103.378 121.666) (end 103.378 68.326) (angle 90) (layer Edge.Cuts) (width 0.15))
